File: Eagle/untitled.brd (EAGLE design)
At the start: 25.4 x 48.1 mm, 26 parts, among them T1 IRLML2502, T2 IRLML2502, T4 IRLML2502

Commit message: Add description nominal of resistors
Parts:
- JP1: value (none) -> CONTROL RING
- JP2: value (none) -> UP RECEIVER
- JP3: value (none) -> PUSH OPEN BUTTON
- JP4: value (none) -> DETECT CALL
- R1, R15: value (none) -> 300
- R16, R17, R18, R3, R5, R7: value (none) -> 10k
- R2, R4, R6: value (none) -> 1k
Changed lines of the file:
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@@
 <?xml version="1.0" encoding="utf-8"?>
 <!DOCTYPE eagle SYSTEM "eagle.dtd">
-<eagle version="7.7.0">
+<eagle version="9.5.1">
 <drawing>
 <settings>
 <setting alwaysvectorfont="no"/>
+<setting keepoldvectorfont="yes"/>
 <setting verticaltext="up"/>
 </settings>
@@
 <param name="dpMaxLengthDifference" value="10mm"/>
 <param name="dpGapFactor" value="2.5"/>
-<param name="checkGrid" value="0"/>
 <param name="checkAngle" value="0"/>
 <param name="checkFont" value="1"/>
 <param name="checkRestrict" value="1"/>
+<param name="checkStop" value="0"/>
+<param name="checkValues" value="0"/>
+<param name="checkNames" value="1"/>
+<param name="checkWireStubs" value="1"/>
+<param name="checkPolygonWidth" value="0"/>
 <param name="useDiameter" value="13"/>
 <param name="maxErrors" value="50"/>
@@
 <attribute name="VALUE" x="9.525" y="33.147" size="1.27" layer="28" rot="MR270"/>
 </element>
-<element name="R2" library="rcl" package="R0805" value="" x="12.7" y="31.75" rot="MR270"/>
-<element name="R3" library="rcl" package="R0805" value="" x="10.16" y="30.48" rot="MR270"/>
-<element name="R1" library="rcl" package="R0805" value="" x="7.62" y="17.018" rot="MR180"/>
-<element name="U$5" library="unt" package="PE0140" value="PE0140" x="3.81" y="6.35"/>
-<element name="U$6" library="unt" package="PE0140" value="PE0140" x="3.81" y="16.51"/>
-<element name="JP1" library="unt" package="1X03" value="" x="8.128" y="43.942" smashed="yes">
+<element name="R2" library="rcl" package="R0805" value="1k" x="12.7" y="31.75" smashed="yes" rot="MR270"/>
+<element name="R3" library="rcl" package="R0805" value="10k" x="10.16" y="30.48" smashed="yes" rot="MR270"/>
+<element name="R1" library="rcl" package="R0805" value="300" x="7.62" y="17.018" smashed="yes" rot="MR180"/>
+<element name="U$5" library="unt" package="PE0140" value="PE0140" x="3.81" y="6.35" smashed="yes"/>
+<element name="U$6" library="unt" package="PE0140" value="PE0140" x="3.81" y="16.51" smashed="yes"/>
+<element name="JP1" library="unt" package="1X03" value="CONTROL RING" x="8.128" y="43.942" smashed="yes">
 <attribute name="VALUE" x="4.318" y="40.767" size="1.27" layer="27"/>
 </element>
-<element name="JP2" library="unt" package="1X03" value="" x="17.272" y="43.942" smashed="yes">
+<element name="JP2" library="unt" package="1X03" value="UP RECEIVER" x="17.272" y="43.942" smashed="yes">
 <attribute name="VALUE" x="13.462" y="40.767" size="1.27" layer="27"/>
 </element>
@@
 <attribute name="VALUE" x="19.558" y="32.131" size="1.27" layer="27" ratio="10" rot="R180"/>
 </element>
-<element name="JP3" library="unt" package="1X02" value="" x="8.128" y="38.862" smashed="yes">
+<element name="JP3" library="unt" package="1X02" value="PUSH OPEN BUTTON" x="8.128" y="38.862" smashed="yes">
 <attribute name="VALUE" x="5.588" y="35.687" size="1.27" layer="27"/>
 </element>
-<element name="JP4" library="unt" package="1X02" value="" x="17.272" y="38.862" smashed="yes" rot="R180">
+<element name="JP4" library="unt" package="1X02" value="DETECT CALL" x="17.272" y="38.862" smashed="yes" rot="R180">
 <attribute name="VALUE" x="19.812" y="42.037" size="1.27" layer="27" rot="R180"/>
 </element>
-<element name="R15" library="rcl" package="R0805" value="" x="18.796" y="36.068" rot="MR180"/>
-<element name="R16" library="rcl" package="R0805" value="" x="6.604" y="35.814" rot="MR0"/>
-<element name="R17" library="rcl" package="R0805" value="" x="20.066" y="30.226" rot="MR90"/>
-<element name="R18" library="rcl" package="R0805" value="" x="15.24" y="30.988" rot="MR270"/>
+<element name="R15" library="rcl" package="R0805" value="300" x="18.796" y="36.068" smashed="yes" rot="MR180"/>
+<element name="R16" library="rcl" package="R0805" value="10k" x="6.604" y="35.814" smashed="yes" rot="MR0"/>
+<element name="R17" library="rcl" package="R0805" value="10k" x="20.066" y="30.226" smashed="yes" rot="MR90"/>
+<element name="R18" library="rcl" package="R0805" value="10k" x="15.24" y="30.988" smashed="yes" rot="MR270"/>
 <element name="T1" library="unt" package="SOT23" value="IRLML2502" x="7.366" y="11.684" smashed="yes" rot="MR270">
 <attribute name="VALUE" x="10.541" y="13.589" size="1.27" layer="28" rot="MR270"/>
 </element>
-<element name="R4" library="rcl" package="R0805" value="" x="14.478" y="12.7" rot="MR0"/>
-<element name="R5" library="rcl" package="R0805" value="" x="10.922" y="11.684" rot="MR270"/>
+<element name="R4" library="rcl" package="R0805" value="1k" x="14.478" y="12.7" smashed="yes" rot="MR0"/>
+<element name="R5" library="rcl" package="R0805" value="10k" x="10.922" y="11.684" smashed="yes" rot="MR270"/>
 <element name="T2" library="unt" package="SOT23" value="IRLML2502" x="7.112" y="21.59" smashed="yes" rot="MR270">
 <attribute name="VALUE" x="10.287" y="23.495" size="1.27" layer="28" rot="MR270"/>
 </element>
-<element name="R6" library="rcl" package="R0805" value="" x="14.478" y="22.606" rot="MR0"/>
-<element name="R7" library="rcl" package="R0805" value="" x="10.922" y="21.59" rot="MR270"/>
+<element name="R6" library="rcl" package="R0805" value="1k" x="14.478" y="22.606" smashed="yes" rot="MR0"/>
+<element name="R7" library="rcl" package="R0805" value="10k" x="10.922" y="21.59" smashed="yes" rot="MR270"/>
 <element name="D1" library="unt" package="DO-214AC" value="1N4007" x="9.398" y="3.048" smashed="yes">
 <attribute name="MPN" value="1N4007" x="9.398" y="3.048" size="1.27" layer="27" display="off"/>
@@
 </signal>
 </signals>
+<mfgpreviewcolors>
+<mfgpreviewcolor name="soldermaskcolor" color="0xC8008000"/>
+<mfgpreviewcolor name="silkscreencolor" color="0xFFFEFEFE"/>
+<mfgpreviewcolor name="backgroundcolor" color="0xFF282828"/>
+<mfgpreviewcolor name="coppercolor" color="0xFFFFBF00"/>
+<mfgpreviewcolor name="substratecolor" color="0xFF786E46"/>
+</mfgpreviewcolors>
 </board>
 </drawing>
